File: BLEVibrator/Hardware/PCB/StrokeRehabilitation.sch (KiCad schematic (older format))
At the start: 30 parts, among them CON1 USB-MICRO-B, P1 CONN_01X01, P2 Programming Header, Q1 MOS_P, Q2 MOSFET_N, SW1 SWITCH_INV, U1 MCP73833, U2 TPS73701_DRV_6, U3 RFD22301, U4 Brushed_DC_motor

Commit message: Added manufacturer part numbers to parts in schematic. Generated a BOM in KiCAD and a rough costing (US-based) using KiCost
Parts:
- BT1: kicost:Kitronik:link (none) -> https://www.kitronik.co.uk/2209-polymer-lithium-ion-battery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
- C1, C2: manf# (none) -> GRM21BR71C105KA01L
- C3: manf# (none) -> GRM21BR61C106KE15L
- C4: manf# (none) -> C0805C101J5GACTU
- C5: manf# (none) -> C1608X7R1E104K080AA
- CON1: manf# (none) -> 10118192-0001LF
- D1, D3: manf# (none) -> SM1204BC-R/G
- D2, D4: manf# (none) -> PMEG2015EH
- Q1: manf# (none) -> SI2367DS-T1-GE3
- Q2: manf# (none) -> MCH3479-TL-H
- R1, R2, R6, R7: manf# (none) -> RC0805FR-07330RL
- R10: manf# (none) -> CRCW06032M20FKEA
- R3: manf# (none) -> RC0805FR-074K99L
- R4: manf# (none) -> RC0805FR-0710KL
- R5, R8: manf# (none) -> RC0805FR-0749K9L
- R9: manf# (none) -> CRCW060310M0FKEA
- SW1: manf# (none) -> SSSS810701
- U1: manf# (none) -> MCP73833T-FCI/MF
- U2: manf# (none) -> TPS73733DRVR
- U3: manf# (none) -> RFD22301
- U4: kicost:PrecisionMicrodrives:link (none) -> https://www.precisionmicrodrives.com/product/307-103-9mm-vi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; manf# (none) -> 307-103
Changed lines of the file:
@@
 F 2 "IainPersonalLibrary:MCPH3_SOT-323" H 9850 2050 60  0001 C CNN
 F 3 "" H 9850 2050 60  0000 C CNN
+F 4 "MCH3479-TL-H" H 9850 2050 60  0001 C CNN "manf#"
 	1    9850 2050
 	1    0    0    -1
@@
 F 2 "IainPersonalLibrary:Yageo_resistor_SMD_0805_reflow" V 9330 2400 50  0001 C CNN
 F 3 "" H 9400 2400 50  0000 C CNN
+F 4 "RC0805FR-0749K9L" H 9400 2400 60  0001 C CNN "manf#"
 	1    9400 2400
 	1    0    0    -1
@@
 F 2 "IainPersonalLibrary:Murata_capacitor_SMD_0805_reflow" H 9538 1200 50  0001 C CNN
 F 3 "" H 9500 1350 50  0000 C CNN
+F 4 "C0805C101J5GACTU" H 9500 1350 60  0001 C CNN "manf#"
 	1    9500 1350
 	1    0    0    -1
@@
 F 2 "IainPersonalLibrary:WireToBoard_1x2_TensionRelief" H 9950 1350 60  0001 C CNN
 F 3 "" H 9950 1350 60  0000 C CNN
+F 4 "307-103" V 9950 1350 60  0001 C CNN "manf#"
+F 5 "https://www.precisionmicrodrives.com/product/307-103-9mm-vibration-motor-25mm-type" V 9950 1350 60  0001 C CNN "kicost:PrecisionMicrodrives:link"
 	1    9950 1350
 	0    1    1    0
@@
 F 2 "IainPersonalLibrary:Murata_capacitor_SMD_0805_reflow" H 8438 2200 50  0001 C CNN
 F 3 "" H 8400 2350 50  0000 C CNN
+F 4 "GRM21BR61C106KE15L" H 8400 2350 60  0001 C CNN "manf#"
 	1    8400 2350
 	1    0    0    -1
@@
 F 2 "IainPersonalLibrary:RFD22301_RFDuino" H 2400 4900 50  0001 L CNN
 F 3 "" H 2600 4400 60  0000 C CNN
+F 4 "RFD22301" H 2600 4400 60  0001 C CNN "manf#"
 	1    2600 4400
 	-1   0    0    1
@@
 F 2 "IainPersonalLibrary:Yageo_resistor_SMD_0805_reflow" V 4630 4400 50  0001 C CNN
 F 3 "" H 4700 4400 50  0000 C CNN
+F 4 "RC0805FR-07330RL" H 4700 4400 60  0001 C CNN "manf#"
 	1    4700 4400
 	1    0    0    -1
@@
 F 2 "IainPersonalLibrary:Yageo_resistor_SMD_0805_reflow" V 4430 4400 50  0001 C CNN
 F 3 "" H 4500 4400 50  0000 C CNN
+F 4 "RC0805FR-07330RL" H 4500 4400 60  0001 C CNN "manf#"
 	1    4500 4400
 	1    0    0    -1
@@
 F 2 "IainPersonalLibrary:SlideSwitch_SSSS810701" H 6400 2200 50  0001 C CNN
 F 3 "" H 6400 2200 50  0000 C CNN
+F 4 "SSSS810701" H 6400 2200 60  0001 C CNN "manf#"
 	1    6400 2200
 	-1   0    0    1
@@
 F 2 "IainPersonalLibrary:Bi_LED_SM1204BC-RG" H 4600 3900 60  0001 C CNN
 F 3 "" H 4600 3900 60  0000 C CNN
+F 4 "SM1204BC-R/G" V 4600 3900 60  0001 C CNN "manf#"
 	1    4600 3900
 	0    -1   -1   0
@@
 F 2 "IainPersonalLibrary:BatteryCon_WireSolder_0.8mm" V 4800 2390 50  0001 C CNN
 F 3 "" V 4800 2390 50  0000 C CNN
+F 4 "https://www.kitronik.co.uk/2209-polymer-lithium-ion-battery-37v-400mah.html" H 4800 2350 60  0001 C CNN "kicost:Kitronik:link"
 	1    4800 2350
 	1    0    0    -1
@@
 F 2 "IainPersonalLibrary:MCP73833-XXX_MF" H 3300 2200 60  0001 C CNN
 F 3 "" H 3300 2200 60  0000 C CNN
+F 4 "MCP73833T-FCI/MF" H 3300 2200 60  0001 C CNN "manf#"
 	1    3300 2200
 	1    0    0    -1
@@
 F 2 "IainPersonalLibrary:Yageo_resistor_SMD_0805_reflow" V 3830 2600 50  0001 C CNN
 F 3 "" H 3900 2600 50  0000 C CNN
+F 4 "RC0805FR-074K99L" H 3900 2600 60  0001 C CNN "manf#"
 	1    3900 2600
 	1    0    0    -1
@@
 F 2 "IainPersonalLibrary:Yageo_resistor_SMD_0805_reflow" V 2380 2000 50  0001 C CNN
 F 3 "" H 2450 2000 50  0000 C CNN
+F 4 "RC0805FR-07330RL" H 2450 2000 60  0001 C CNN "manf#"
 	1    2450 2000
 	-1   0    0    1
@@
 F 2 "IainPersonalLibrary:Yageo_resistor_SMD_0805_reflow" V 2180 2000 50  0001 C CNN
 F 3 "" H 2250 2000 50  0000 C CNN
+F 4 "RC0805FR-07330RL" H 2250 2000 60  0001 C CNN "manf#"
 	1    2250 2000
 	-1   0    0    1
@@
 F 2 "IainPersonalLibrary:Bi_LED_SM1204BC-RG" H 2350 1500 60  0001 C CNN
 F 3 "" H 2350 1500 60  0000 C CNN
+F 4 "SM1204BC-R/G" V 2350 1500 60  0001 C CNN "manf#"
 	1    2350 1500
 	0    1    -1   0
@@
 F 2 "IainPersonalLibrary:Yageo_resistor_SMD_0805_reflow" V 4080 2600 50  0001 C CNN
 F 3 "" H 4150 2600 50  0000 C CNN
+F 4 "RC0805FR-0710KL" H 4150 2600 60  0001 C CNN "manf#"
 	1    4150 2600
 	1    0    0    -1
@@
 F 2 "IainPersonalLibrary:Murata_capacitor_SMD_0805_reflow" H 1938 1250 50  0001 C CNN
 F 3 "" H 1900 1400 50  0000 C CNN
+F 4 "GRM21BR71C105KA01L" H 1900 1400 60  0001 C CNN "manf#"
 	1    1900 1400
 	1    0    0    -1
@@
 F 2 "IainPersonalLibrary:Vishay_SOT-23" H 5450 1900 60  0001 C CNN
 F 3 "" H 5450 1900 60  0000 C CNN
+F 4 "SI2367DS-T1-GE3" V 5450 1900 60  0001 C CNN "manf#"
 	1    5450 1900
 	0    1    1    0
@@
 F 2 "IainPersonalLibrary:SOD-123F" H 5700 1550 50  0001 C CNN
 F 3 "" H 5700 1550 50  0000 C CNN
+F 4 "PMEG2015EH" V 5700 1550 60  0001 C CNN "manf#"
 	1    5700 1550
 	0    -1   -1   0
@@
 F 2 "IainPersonalLibrary:Yageo_resistor_SMD_0805_reflow" V 5130 1550 50  0001 C CNN
 F 3 "" H 5200 1550 50  0000 C CNN
+F 4 "RC0805FR-0749K9L" H 5200 1550 60  0001 C CNN "manf#"
 	1    5200 1550
 	1    0    0    -1
@@
 F 2 "IainPersonalLibrary:Murata_capacitor_SMD_0805_reflow" H 4488 2200 50  0001 C CNN
 F 3 "" H 4450 2350 50  0000 C CNN
+F 4 "GRM21BR71C105KA01L" H 4450 2350 60  0001 C CNN "manf#"
 	1    4450 2350
 	1    0    0    -1
@@
 F 2 "IainPersonalLibrary:SOD-123F" H 10350 1400 50  0001 C CNN
 F 3 "" H 10350 1400 50  0000 C CNN
+F 4 "PMEG2015EH" V 10350 1400 60  0001 C CNN "manf#"
 	1    10350 1400
 	0    1    1    0
@@
 F 2 "IainPersonalLibrary:TPS73701_DRV_6" H 7170 2430 20  0001 C CNN
 F 3 "" H 7140 2280 60  0000 C CNN
+F 4 "TPS73733DRVR" H 7750 2150 60  0001 C CNN "manf#"
 	1    7750 2150
 	1    0    0    -1
@@
 F 2 "IainPersonalLibrary:Micro_USB_Amphenol_10118192-0001LF" H 1200 1200 50  0001 C CNN
 F 3 "" H 1200 1200 50  0000 C CNN
+F 4 "10118192-0001LF" H 1200 1300 60  0001 C CNN "manf#"
 	1    1200 1300
 	1    0    0    -1
@@
 F 2 "Resistors_SMD:R_0603" V 5530 4550 50  0001 C CNN
 F 3 "" H 5600 4550 50  0000 C CNN
+F 4 "CRCW06032M20FKEA" V 5600 4550 60  0001 C CNN "manf#"
 	1    5600 4550
 	1    0    0    -1
@@
 F 2 "Resistors_SMD:R_0603" V 5530 3950 50  0001 C CNN
 F 3 "" H 5600 3950 50  0000 C CNN
+F 4 "CRCW060310M0FKEA" V 5600 3950 60  0001 C CNN "manf#"
 	1    5600 3950
 	1    0    0    -1
@@
 F 2 "Capacitors_SMD:C_0603" H 5938 4400 50  0001 C CNN
 F 3 "" H 5900 4550 50  0000 C CNN
+F 4 "C1608X7R1E104K080AA" H 5900 4550 60  0001 C CNN "manf#"
 	1    5900 4550
 	1    0    0    -1
