File: BLEVibrator/Hardware/PCB/StrokeRehabilitation.kicad_pcb (KiCad board)
At the start: 2 copper layers, 32 x 48 mm, 30 parts, among them CON1 USB-MICRO-B, P1 CONN_01X01, P2 Programming Header, Q1 MOS_P, Q2 MOSFET_N, SW1 SWITCH_INV, U1 MCP73833, U2 TPS73701_DRV_6, U3 RFD22301, U4 Brushed_DC_motor

Commit message: more clean up of silkscreen label placement
Parts:
- C5: footprint Capacitors_SMD:C_0603 -> IainPersonalLibrary:C_0603
- R10, R9: footprint Resistors_SMD:R_0603 -> IainPersonalLibrary:R_0603
Changed lines of the file:
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@@
       (drillshape 0)
       (scaleselection 1)
-      (outputdirectory ""))
+      (outputdirectory Gerbers/))
   )
   (net 0 "")
@@
   (module IainPersonalLibrary:Micro_USB_Amphenol_10118192-0001LF locked (layer F.Cu)
     (at 165.38 127.0276 90)
-    (fp_text reference CON1 (at 0 5.75 90) (layer F.SilkS)
+    (fp_text reference CON1 (at 0 5.75 90) (layer F.SilkS) hide
       (effects (font (size 1 1) (thickness 0.15)))
     )
@@
   (module IainPersonalLibrary:Vishay_SOT-23 (layer F.Cu)
     (at 161.3668 129.6184 90)
-    (fp_text reference Q1 (at 2.032 -1.2192 180) (layer F.SilkS)
+    (fp_text reference Q1 (at -0.0316 -2.4168 270) (layer F.SilkS)
       (effects (font (size 1 1) (thickness 0.15)))
     )
@@
   (module IainPersonalLibrary:TPS73701_DRV_6 (layer F.Cu)
     (at 158.05972 132.09744 270)
-    (fp_text reference U2 (at -2.22504 -0.00508 360) (layer F.SilkS)
+    (fp_text reference U2 (at 2.15256 0.00972 360) (layer F.SilkS)
       (effects (font (size 1 1) (thickness 0.15)))
     )
@@
       (net 1 VDD))
   )
-  (module Capacitors_SMD:C_0603 (layer F.Cu)
-    (at 164.25 119.9 270)
-    (descr "Capacitor SMD 0603, reflow soldering, AVX (see smccp.pdf)")
-    (tags "capacitor 0603")
-    (attr smd)
-    (fp_text reference C5 (at 0 5.35 270) (layer F.SilkS)
-      (effects (font (size 1 1) (thickness 0.15)))
-    )
-    (fp_text value 100n (at 0 1.9 270) (layer F.Fab) hide
-      (effects (font (size 1 1) (thickness 0.15)))
-    )
-    (fp_line (start -1.45 -0.75) (end 1.45 -0.75) (layer F.CrtYd) (width 0.05))
-    (fp_line (start -1.45 0.75) (end 1.45 0.75) (layer F.CrtYd) (width 0.05))
-    (fp_line (start -1.45 -0.75) (end -1.45 0.75) (layer F.CrtYd) (width 0.05))
-    (fp_line (start 1.45 -0.75) (end 1.45 0.75) (layer F.CrtYd) (width 0.05))
-    (fp_line (start -0.35 -0.6) (end 0.35 -0.6) (layer F.SilkS) (width 0.15))
-    (fp_line (start 0.35 0.6) (end -0.35 0.6) (layer F.SilkS) (width 0.15))
-    (pad 1 smd rect (at -0.75 0 270) (size 0.8 0.75) (layers F.Cu F.Paste F.Mask)
-      (net 30 BatteryLevel))
-    (pad 2 smd rect (at 0.75 0 270) (size 0.8 0.75) (layers F.Cu F.Paste F.Mask)
-      (net 2 GND))
-    (model Capacitors_SMD.3dshapes/C_0603.wrl
-      (at (xyz 0 0 0))
-      (scale (xyz 1 1 1))
-      (rotate (xyz 0 0 0))
-    )
-  )
-  (module Resistors_SMD:R_0603 (layer F.Cu)
+  (module IainPersonalLibrary:TestPoint_SMD_1x1 (layer F.Cu)
+    (at 140.85 107.6)
+    (fp_text reference P1 (at 2 9.3) (layer F.SilkS)
+      (effects (font (size 1 1) (thickness 0.15)))
+    )
+    (fp_text value CONN_01X01 (at 0.05 -3.6) (layer F.Fab) hide
+      (effects (font (size 1 1) (thickness 0.15)))
+    )
+    (pad 1 smd rect (at 0 0) (size 1.6 1.6) (layers F.Cu F.Mask)
+      (net 31 "Net-(P1-Pad1)"))
+  )
+  (module IainPersonalLibrary:R_0603 (layer F.Cu)
     (at 160.3 119.9 90)
     (descr "Resistor SMD 0603, reflow soldering, Vishay (see dcrcw.pdf)")
     (tags "resistor 0603")
     (attr smd)
-    (fp_text reference R9 (at 0 -3.95 90) (layer F.SilkS)
+    (fp_text reference R9 (at 0 -4.15 90) (layer F.SilkS)
       (effects (font (size 1 1) (thickness 0.15)))
     )
@@
     (fp_line (start -1.3 -0.8) (end -1.3 0.8) (layer F.CrtYd) (width 0.05))
     (fp_line (start 1.3 -0.8) (end 1.3 0.8) (layer F.CrtYd) (width 0.05))
-    (fp_line (start 0.5 0.675) (end -0.5 0.675) (layer F.SilkS) (width 0.15))
-    (fp_line (start -0.5 -0.675) (end 0.5 -0.675) (layer F.SilkS) (width 0.15))
     (pad 1 smd rect (at -0.75 0 90) (size 0.5 0.9) (layers F.Cu F.Paste F.Mask)
       (net 10 +BATT))
@@
     )
   )
-  (module Resistors_SMD:R_0603 (layer F.Cu)
+  (module IainPersonalLibrary:C_0603 (layer F.Cu)
+    (at 164.25 119.9 270)
+    (descr "Capacitor SMD 0603, reflow soldering, AVX (see smccp.pdf)")
+    (tags "capacitor 0603")
+    (attr smd)
+    (fp_text reference C5 (at 0 5.35 270) (layer F.SilkS)
+      (effects (font (size 1 1) (thickness 0.15)))
+    )
+    (fp_text value 100n (at 0 1.9 270) (layer F.Fab) hide
+      (effects (font (size 1 1) (thickness 0.15)))
+    )
+    (fp_line (start -1.45 -0.75) (end 1.45 -0.75) (layer F.CrtYd) (width 0.05))
+    (fp_line (start -1.45 0.75) (end 1.45 0.75) (layer F.CrtYd) (width 0.05))
+    (fp_line (start -1.45 -0.75) (end -1.45 0.75) (layer F.CrtYd) (width 0.05))
+    (fp_line (start 1.45 -0.75) (end 1.45 0.75) (layer F.CrtYd) (width 0.05))
+    (pad 1 smd rect (at -0.75 0 270) (size 0.8 0.75) (layers F.Cu F.Paste F.Mask)
+      (net 30 BatteryLevel))
+    (pad 2 smd rect (at 0.75 0 270) (size 0.8 0.75) (layers F.Cu F.Paste F.Mask)
+      (net 2 GND))
+    (model Capacitors_SMD.3dshapes/C_0603.wrl
+      (at (xyz 0 0 0))
+      (scale (xyz 1 1 1))
+      (rotate (xyz 0 0 0))
+    )
+  )
+  (module IainPersonalLibrary:R_0603 (layer F.Cu)
     (at 162.3 119.9 270)
     (descr "Resistor SMD 0603, reflow soldering, Vishay (see dcrcw.pdf)")
     (tags "resistor 0603")
     (attr smd)
-    (fp_text reference R10 (at 0 4.65 270) (layer F.SilkS)
+    (fp_text reference R10 (at 0 4.85 270) (layer F.SilkS)
       (effects (font (size 1 1) (thickness 0.15)))
     )
@@
     (fp_line (start -1.3 -0.8) (end -1.3 0.8) (layer F.CrtYd) (width 0.05))
     (fp_line (start 1.3 -0.8) (end 1.3 0.8) (layer F.CrtYd) (width 0.05))
-    (fp_line (start 0.5 0.675) (end -0.5 0.675) (layer F.SilkS) (width 0.15))
-    (fp_line (start -0.5 -0.675) (end 0.5 -0.675) (layer F.SilkS) (width 0.15))
     (pad 1 smd rect (at -0.75 0 270) (size 0.5 0.9) (layers F.Cu F.Paste F.Mask)
       (net 30 BatteryLevel))
@@
     )
   )
-  (module IainPersonalLibrary:TestPoint_SMD_1x1 (layer F.Cu)
-    (at 140.85 107.6)
-    (fp_text reference P1 (at 2 9.3) (layer F.SilkS)
-      (effects (font (size 1 1) (thickness 0.15)))
-    )
-    (fp_text value CONN_01X01 (at 0.05 -3.6) (layer F.Fab) hide
-      (effects (font (size 1 1) (thickness 0.15)))
-    )
-    (pad 1 smd rect (at 0 0) (size 1.6 1.6) (layers F.Cu F.Mask)
-      (net 31 "Net-(P1-Pad1)"))
-  )
   (gr_text "BLEVibrator v0.3\nDesigned by Iain Chalmers\nhttps://github.com/icchalmers/Sit-To-Stand" (at 149.65 122.2 90) (layer B.SilkS)
